File: board/t80-rs232.kicad_pcb (KiCad board)
At the start: 2 copper layers, 40 x 80 mm, 25 parts, among them J1 8P8C, U1 ATSAMD09C13A-SS, U2 MAX232

Commit message: WIP
Parts:
- removed JP3: BOOT, Jumper:SolderJumper-2_P1.3mm_Open_Pad1.0x1.5mm
- removed NT1, NT2, NT3, NT4: NetTie_2, t80:NetTie-2mm-T80
- removed X3: ~, Connector_PinHeader_2.54mm:PinHeader_2x05_P2.54mm_Vertical
- added X1: SWD, Drake:SWD, F.Cu at (136.0, 92.2)
- X2: footprint Connector_PinHeader_2.54mm:PinHeader_2x05_P2.54mm_Vertical -> Connector_IDC:IDC-Header_2x04_P2.54mm_Vertical
- moved C7 73.1 mm to (124.0, 50.2), turned to 180 degrees
- moved C5 69.8 mm to (128.0, 50.2), turned to 180 degrees
- moved C4 68.9 mm to (132.0, 50.2), turned to 180 degrees
- moved R2 68.0 mm to (126.0, 65.2), turned to 180 degrees
- moved C1 64.8 mm to (131.0, 65.2)
- moved C6 64.2 mm to (135.0, 57.2), turned to -90 degrees
- moved R4 63.0 mm to (126.0, 67.2)
- moved U2 61.0 mm to (128.0, 57.2), turned to -90 degrees
- moved R5 55.6 mm to (132.0, 100.2)
- moved C3 55.5 mm to (131.0, 67.2)
- moved R1 52.2 mm to (124.0, 103.2), turned to -90 degrees
- moved R3 51.5 mm to (126.5, 103.2), turned to -90 degrees
- moved D1 50.9 mm to (132.0, 103.2)
- moved U1 49.8 mm to (132.0, 79.2)
- moved C2 46.3 mm to (137.0, 78.2), turned to 90 degrees
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Connections:
- X2 pad 1: /PWR_LINE_12V -> GND
- X2 pad 2: /PWR_LINE_12V -> /SCL
- X2 pad 3: /PWR_LINE_GND -> /SDA
- X2 pad 4: /PWR_LINE_GND -> +3V3
- X2 pad 5: /SCL -> /RST
- X2 pad 6: /SDA -> /IRQ
- X2 pad 7: /RST -> GND
- X2 pad 8: /IRQ -> +5V
Routing:
- net /PWR_LINE_GND: track 58.4 -> 0.00 mm, vias 7 -> 0
- net Net-(U2-T1OUT): track 0.00 -> 57.4 mm
- net Net-(U2-R1IN): track 0.00 -> 55.5 mm
- net +5V: track 0.00 -> 42.7 mm, vias 0 -> 2
- net /PWR_LINE_5V: track 38.0 -> 0.00 mm, vias 1 -> 0
- net /PWR_LINE_3V3: track 38.0 -> 0.00 mm
- net /PWR_LINE_12V: track 37.4 -> 0.00 mm
- net +3V3: track 0.00 -> 32.0 mm, vias 0 -> 3
- net /SCL: track 35.8 -> 6.08 mm, vias 1 -> 0
- net GND: track 0.00 -> 25.8 mm, vias 0 -> 7
- net /RST: track 35.8 -> 10.2 mm, vias 1 -> 0
- net /LED: track 0.00 -> 25.4 mm
- net /SDA: track 35.8 -> 11.7 mm
- net /TX_3V: track 0.00 -> 24.2 mm
- net /SWCLK: track 0.00 -> 23.0 mm
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Other:
- board size 40 x 80 mm -> 20 x 80 mm
- board text added: "T80-RS232 v1.0"
- board text removed: "T80-Template v1.0"
- board text removed: "connector screws"

Commit message: WIP
Parts:
- U2: footprint Package_SO:SO-16_5.3x10.2mm_P1.27mm -> Package_SO:SOIC-16W_5.3x10.2mm_P1.27mm
- moved D1 50.9 mm to (120.0, 53.8), turned to -90 degrees
- moved R5 41.8 mm to (120.0, 60.2), turned to 90 degrees
- moved R1 3.91 mm to (121.0, 105.8), turned to 0 degrees
- moved R3 2.92 mm to (125.0, 105.8), turned to 180 degrees
- moved X1 2.00 mm to (136.0, 90.2)
Routing:
- net /LED: track 25.4 -> 71.6 mm, vias 0 -> 2
- net /RX_RS232: track 12.5 -> 5.65 mm
- net /TX_RS232: track 4.72 -> 8.37 mm
- net Net-(U2-T1OUT): track 57.4 -> 60.9 mm
- net Net-(U2-R1IN): track 55.5 -> 58.8 mm
- net /SWDIO: track 7.28 -> 5.28 mm
- net GND: track 25.8 -> 27.7 mm, vias 7 -> 6
- net /SWCLK: track 23.0 -> 24.6 mm
- net Net-(D1-A): track 3.01 -> 4.48 mm
- net +5V: track 42.7 -> 42.0 mm
Other:
- board text added: "0 1 2 3 4 5 6 7 8"
