File: board/t80-rs232.kicad_pcb (KiCad board)
At the start: 2 copper layers, 20 x 80 mm, 20 parts, among them J1 8P8C, U1 ATSAMD09C13A-SS, U2 MAX232, X1 SWD

Commit message: WIP
Parts:
- removed J1: 8P8C, Connector_RJ:RJ45_Amphenol_54602-x08_Horizontal
- added J2: RS232, Drake:DG235-3.81-03P, F.Cu at (124.2, 114.3)
Routing:
- net /TX_RS232: track 8.37 -> 21.8 mm
- net /RX_RS232: track 5.65 -> 15.2 mm
Other:
- board text added: "GND"
- board text added: "RX"
- board text added: "TX"

Commit message: WIP
Parts:
- J2: value RS232 -> RS485
Connections:
- net /RX_RS232 renamed /RX_RS485
- net /TX_RS232 renamed /TX_RS485
Other:
- board text added: "T80-RS485 v1.0"
- board text removed: "T80-RS232 v1.0"
