File: board/t80-rs232.kicad_sch (KiCad schematic)
At the start: 26 parts, among them J1 8P8C, U1 MAX232, U2 ATSAMD09C13A-SS, X3 SWD

Commit message: WIP
Parts:
- removed JP3: BOOT, symbol Jumper:SolderJumper_2_Open
- removed NT1 (x4): NetTie_2, symbol Device:NetTie_2
- removed X1 (x2): ~, symbol t80:t80-pin-header
- added X1: ~, symbol t80:t80-pin-header
Connections:
- net +3V3: now also X1.4 (3V3)
- net +5V: now also X1.8 (5V)
- net GND: now also X1.1 (GND), X1.7 (GND)
- net IRQ: now also X1.6 (IRQ)
- net RST: now also X1.5 (RST)
- net SCL: now also X1.2 (SCL)
- net SDA: now also X1.3 (SDA)
- no-connect marks 9 -> 10

Commit message: WIP
Parts:
- removed J1: 8P8C, Connector_RJ:RJ45_Amphenol_54602-x08_Horizontal, symbol Connector:8P8C
- added J2: RS232, symbol Connector:Conn_01x03_Female
Connections:
- net GND: now also J2.1 (Pin_1)
- net RX_RS232: now also J2.2 (Pin_2)
- net TX_RS232: now also J2.3 (Pin_3)
- no-connect marks 10 -> 5
Changed lines of the file:
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@@
   (no_connect (at 203.2 77.47))
   (no_connect (at 203.2 87.63))
-  (no_connect (at 233.68 128.27))
-  (no_connect (at 233.68 120.65))
-  (no_connect (at 233.68 123.19))
-  (no_connect (at 233.68 125.73))
-  (no_connect (at 233.68 118.11))
   (no_connect (at 115.57 66.04))
   (no_connect (at 162.56 87.63))
@@
     (effects (font (size 1.27 1.27)) (justify left bottom))
   )
-  (label "RX_RS232" (at 233.68 113.03 180) (fields_autoplaced)
+  (label "RX_RS232" (at 186.69 128.27 180) (fields_autoplaced)
     (effects (font (size 1.27 1.27)) (justify right bottom))
   )
@@
     (effects (font (size 1.27 1.27)) (justify right bottom))
   )
-  (label "TX_RS232" (at 233.68 115.57 180) (fields_autoplaced)
+  (label "TX_RS232" (at 186.69 125.73 180) (fields_autoplaced)
     (effects (font (size 1.27 1.27)) (justify right bottom))
   )
@@
     (pin "2")
   )
-  (symbol (lib_id "power:GND") (at 233.68 130.81 0) (unit 1)
-    (in_bom yes) (on_board yes) (dnp no) (fields_autoplaced)
-    (default_instance (reference "#PWR?") (unit 1) (value "GND") (footprint ""))
-    (property "Reference" "#PWR?" (id 0) (at 233.68 137.16 0)
-      (effects (font (size 1.27 1.27)) hide)
-    )
-    (property "Value" "GND" (id 1) (at 233.68 134.8661 0)
-      (effects (font (size 1.27 1.27)))
-    )
-    (property "Footprint" "" (id 2) (at 233.68 130.81 0)
-      (effects (font (size 1.27 1.27)) hide)
-    )
-    (property "Datasheet" "" (id 3) (at 233.68 130.81 0)
+  (symbol (lib_id "power:GND") (at 186.69 130.81 0) (unit 1)
+    (in_bom yes) (on_board yes) (dnp no) (fields_autoplaced)
+    (default_instance (reference "#PWR?") (unit 1) (value "GND") (footprint ""))
+    (property "Reference" "#PWR?" (id 0) (at 186.69 137.16 0)
+      (effects (font (size 1.27 1.27)) hide)
+    )
+    (property "Value" "GND" (id 1) (at 186.69 134.8661 0)
+      (effects (font (size 1.27 1.27)))
+    )
+    (property "Footprint" "" (id 2) (at 186.69 130.81 0)
+      (effects (font (size 1.27 1.27)) hide)
+    )
+    (property "Datasheet" "" (id 3) (at 186.69 130.81 0)
       (effects (font (size 1.27 1.27)) hide)
     )
@@
     (pin "2")
   )
+  (symbol (lib_id "Connector:Conn_01x03_Female") (at 191.77 128.27 0) (mirror x) (unit 1)
+    (in_bom yes) (on_board yes) (dnp no)
+    (default_instance (reference "J2") (unit 1) (value "RS232") (footprint ""))
+    (property "Reference" "J2" (id 0) (at 192.4812 128.8645 0)
+      (effects (font (size 1.27 1.27)) (justify left))
+    )
+    (property "Value" "RS232" (id 1) (at 192.4812 127.1023 0)
+      (effects (font (size 1.27 1.27)) (justify left))
+    )
+    (property "Footprint" "" (id 2) (at 191.77 128.27 0)
+      (effects (font (size 1.27 1.27)) hide)
+    )
+    (property "Datasheet" "~" (id 3) (at 191.77 128.27 0)
+      (effects (font (size 1.27 1.27)) hide)
+    )
+    (pin "1")
+    (pin "2")
+    (pin "3")
+  )
   (symbol (lib_id "power:GND") (at 147.32 92.71 0) (unit 1)
     (in_bom yes) (on_board yes) (dnp no) (fields_autoplaced)
@@
     (pin "1")
   )
-  (symbol (lib_id "Connector:8P8C") (at 243.84 120.65 180) (unit 1)
-    (in_bom yes) (on_board yes) (dnp no) (fields_autoplaced)
-    (default_instance (reference "J1") (unit 1) (value "8P8C") (footprint "Connector_RJ:RJ45_Amphenol_54602-x08_Horizontal"))
-    (property "Reference" "J1" (id 0) (at 252.222 121.3255 0)
-      (effects (font (size 1.27 1.27)) (justify right))
-    )
-    (property "Value" "8P8C" (id 1) (at 252.222 123.0877 0)
-      (effects (font (size 1.27 1.27)) (justify right))
-    )
-    (property "Footprint" "Connector_RJ:RJ45_Amphenol_54602-x08_Horizontal" (id 2) (at 243.84 121.285 90)
-      (effects (font (size 1.27 1.27)) hide)
-    )
-    (property "Datasheet" "~" (id 3) (at 243.84 121.285 90)
-      (effects (font (size 1.27 1.27)) hide)
-    )
-    (pin "1")
-    (pin "2")
-    (pin "3")
-    (pin "4")
-    (pin "5")
-    (pin "6")
-    (pin "7")
-    (pin "8")
-  )
   (symbol (lib_id "Device:R") (at 223.52 72.39 90) (unit 1)
     (in_bom yes) (on_board yes) (dnp no) (fields_autoplaced)
@@
       (reference "D1") (unit 1) (value "LED") (footprint "LED_SMD:LED_0805_2012Metric_Pad1.15x1.40mm_HandSolder")
     )
-    (path "/fcbcf2a1-c077-4ea2-be23-bee79fbee537"
-      (reference "J1") (unit 1) (value "8P8C") (footprint "Connector_RJ:RJ45_Amphenol_54602-x08_Horizontal")
+    (path "/e7e00e60-a697-4567-a364-e0f9c8ed95db"
+      (reference "J2") (unit 1) (value "RS232") (footprint "Drake:DG235-3.81-03P")
     )
     (path "/efc8e824-00c2-4eb7-b6ad-b59df64753cb"

Commit message: WIP
Parts:
- J2: value RS232 -> RS485
Connections:
- net RX_RS232 renamed RX_RS485
- net TX_RS232 renamed TX_RS485
Changed lines of the file:
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@@
     (effects (font (size 1.27 1.27)) (justify right bottom))
   )
-  (label "TX_RS232" (at 229.87 72.39 0) (fields_autoplaced)
+  (label "TX_RS485" (at 229.87 72.39 0) (fields_autoplaced)
     (effects (font (size 1.27 1.27)) (justify left bottom))
   )
@@
     (effects (font (size 1.27 1.27)) (justify left bottom))
   )
-  (label "RX_RS232" (at 186.69 128.27 180) (fields_autoplaced)
+  (label "RX_RS485" (at 186.69 128.27 180) (fields_autoplaced)
     (effects (font (size 1.27 1.27)) (justify right bottom))
   )
@@
     (effects (font (size 1.27 1.27)) (justify right bottom))
   )
-  (label "TX_RS232" (at 186.69 125.73 180) (fields_autoplaced)
+  (label "TX_RS485" (at 186.69 125.73 180) (fields_autoplaced)
     (effects (font (size 1.27 1.27)) (justify right bottom))
   )
@@
     (effects (font (size 1.27 1.27)) (justify left bottom))
   )
-  (label "RX_RS232" (at 229.87 82.55 0) (fields_autoplaced)
+  (label "RX_RS485" (at 229.87 82.55 0) (fields_autoplaced)
     (effects (font (size 1.27 1.27)) (justify left bottom))
   )
@@
   (symbol (lib_id "Connector:Conn_01x03_Female") (at 191.77 128.27 0) (mirror x) (unit 1)
     (in_bom yes) (on_board yes) (dnp no)
-    (default_instance (reference "J2") (unit 1) (value "RS232") (footprint ""))
+    (default_instance (reference "J2") (unit 1) (value "RS485") (footprint ""))
     (property "Reference" "J2" (id 0) (at 192.4812 128.8645 0)
       (effects (font (size 1.27 1.27)) (justify left))
     )
-    (property "Value" "RS232" (id 1) (at 192.4812 127.1023 0)
+    (property "Value" "RS485" (id 1) (at 192.4812 127.1023 0)
       (effects (font (size 1.27 1.27)) (justify left))
     )
@@
     )
     (path "/e7e00e60-a697-4567-a364-e0f9c8ed95db"
-      (reference "J2") (unit 1) (value "RS232") (footprint "Drake:DG235-3.81-03P")
+      (reference "J2") (unit 1) (value "RS485") (footprint "Drake:DG235-3.81-03P")
     )
     (path "/efc8e824-00c2-4eb7-b6ad-b59df64753cb"
