File: board/t80-rs485.kicad_sch (KiCad schematic)
At the start: 20 parts, among them J2 RS485, U1 MAX232, U2 ATSAMD09C13A-SS, X3 SWD

Commit message: WIP
Parts:
- removed C1 (x4): C, Capacitor_SMD:C_0805_2012Metric_Pad1.18x1.45mm_HandSolder, symbol Device:C
- removed JP1: A1, symbol Jumper:SolderJumper_3_Open
- removed R1 (x3): 270R, Resistor_SMD:R_0805_2012Metric_Pad1.20x1.40mm_HandSolder, symbol Device:R
- removed U1: MAX232, symbol Interface_UART:MAX232
- added U3: ST3485EBD, Package_SO:SOIC-8_3.9x4.9mm_P1.27mm, symbol Interface_UART:ST485EBDR
- C1: value C -> 1u
- C2, C3: renamed from C1; value C -> 100n
- D1: footprint (none) -> LED_SMD:LED_0805_2012Metric_Pad1.15x1.40mm_HandSolder
- J2: footprint (none) -> Drake:DG235-3.81-03P
- JP1: footprint (none) -> Jumper:SolderJumper-3_P2.0mm_Open_TrianglePad1.0x1.5mm
- R1: value 270R -> 120R
- X1: renamed from X3; footprint drake:SWD -> Drake:SWD
- X2: renamed from X1; footprint (none) -> Connector_IDC:IDC-Header_2x04_P2.54mm_Vertical
- renumbered R1 to R5, U2 to U1
Connections:
- net A2 is gone; now on net ADDR: U1.3 (PA09/XOUT)
- net RX_RS485 is gone; now on net RS485_A: J2.2 (Pin_2)
- net +3V3: now also C1.2, C3.2, U3.8 (VCC)
- net +5V: no longer C1.2, C3.2
- net GND: now also U3.5 (GND)
- net RS485_A: now reaches R1.1
- net RS485_A: now also U3.6 (A)
- net A1 renamed ADDR
- net ADDR: no longer U1.2 (PA08/XIN)
- net RX_3V renamed RX
- net RX: now also U3.1 (RO)
- net TX_3V renamed TX
- net TX: now also U3.4 (DI)
- net TX_RS485 renamed RS485_B
- net RS485_B: now also U3.7 (B)
- new net TXE: U1.2 (PA08/XIN), U3.2 (~{RE}), U3.3 (DE)
- no-connect marks 5 -> 1
Other:
- moved on the sheet: C1, C3, R1
